File: usb_hub.kicad_pcb (KiCad board)
At the start: 4 copper layers, 100 x 60 mm, 80 parts, among them J1 USB_C_Receptacle_USB2.0_16P, J2 USB_C_Receptacle_USB2.0_16P, J3 USB_C_Receptacle_USB2.0_16P, J4 USB_A, J5 USB_A, J7 Conn_01x04_Pin, J8 Conn_01x04_Pin, SW1 SW_SPDT, U1 USB2514B_Bi, U10 STM32F103C8T6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

Commit message: Significant work on pcb again
Parts:
- added G***: LOGO, LOGO, F.Cu at (174.5, 110.0)
- moved R12 6.00 mm to (141.5, 85.0), turned to 0 degrees
- moved R13 5.75 mm to (135.8, 85.0), turned to 180 degrees
- moved C3 1.79 mm to (148.5, 98.5)
- moved C23 1.13 mm to (110.2, 115.0), turned to -90 degrees
- moved C11 0.96 mm to (141.4, 104.6)
- moved C20 0.95 mm to (142.8, 105.7)
- moved R15 0.71 mm to (146.5, 110.0), turned to 0 degrees
- moved C6 0.20 mm to (153.3, 108.5)
- moved R14 0.20 mm to (152.3, 108.5)
Connections:
- U10 pad 21: /OCS_N3 -> unconnected-(U10-PB10-Pad21)
- U10 pad 22: /OCS_N4 -> unconnected-(U10-PB11-Pad22)
- U10 pad 31: unconnected-(U10-PA10-Pad31) -> /OCS_N3
- U10 pad 32: unconnected-(U10-PA11-Pad32) -> /OCS_N4
- U10 pad 39: unconnected-(U10-PB3-Pad39) -> /OCS_N2
- U10 pad 40: unconnected-(U10-PB4-Pad40) -> /OCS_N1
- U10 pad 45: /OCS_N1 -> unconnected-(U10-PB8-Pad45)
- U10 pad 46: /OCS_N2 -> unconnected-(U10-PB9-Pad46)
Routing:
- net VBUS: track 35.8 -> 255.0 mm, vias 7 -> 10
- net /OCS_N2: track 0.00 -> 76.3 mm, vias 0 -> 5
- net /EN1: track 0.00 -> 65.3 mm, vias 0 -> 3
- net /OCS_N1: track 0.00 -> 62.3 mm, vias 0 -> 3
- net /EN2: track 0.00 -> 54.8 mm, vias 0 -> 4
- net /EN4: track 0.00 -> 42.8 mm, vias 0 -> 2
- net /OCS_N4: track 0.00 -> 40.4 mm, vias 0 -> 3
- net /OCS_N3: track 0.00 -> 39.3 mm, vias 0 -> 4
- net /EN3: track 0.00 -> 39.2 mm, vias 0 -> 3
- net /LED_DATA: track 0.00 -> 34.4 mm, vias 0 -> 4
- net +3V3: track 36.8 -> 48.0 mm, vias 21 -> 30
- net Net-(J3-CC1): track 0.00 -> 3.38 mm
- net Net-(J2-CC1): track 0.00 -> 3.38 mm
- net Net-(J3-CC2): track 0.00 -> 3.22 mm
- net Net-(J2-CC2): track 0.00 -> 3.12 mm
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- added copper zone on In2.Cu, net +3V3
- added copper zone on F.Cu, net GND
- added copper zone on In1.Cu, net GND
Other:
- board text added: "L Cooke | 4²/3²/45²"
- board text added: "STM32F103C8T6"
- board text added: "TWO Type-C Ports TWO Type-A Ports"
- board text added: "USB 2.0 FS Hub"
- board text added: "USB2514Bi"

Commit message: Board finished, sending out for fab
Parts:
- added SW2: SW_Push, libs:SW-SMD_L3.9-W3.0-P4.45, F.Cu at (122.8, 122.2)
- moved C20 0.84 mm to (142.0, 105.7)
Routing:
- net /NRST: track 8.82 -> 21.2 mm, vias 2 -> 5
- net VBUS_1: track 24.6 -> 35.6 mm, vias 2 -> 3
- net VBUS_2: track 24.9 -> 35.2 mm
- net VBUS_3: track 24.0 -> 34.0 mm
- net VBUS_4: track 17.1 -> 26.7 mm
- net GND: track 32.9 -> 38.5 mm, vias 239 -> 248
- net +3V3: track 48.0 -> 50.6 mm, vias 30 -> 32
- net VBUS: vias 10 -> 9
Other:
- board text added: "BOOT"
- board text added: "RESET"
