File: usb_hub.kicad_sch (KiCad schematic)
At the start: 14 parts, among them J1 USB_C_Receptacle_USB2.0_16P, J2 USB_C_Receptacle_USB2.0_16P, J3 USB_C_Receptacle_USB2.0_16P, J4 USB_A, U1 USB2514B_Bi, U2 AMS1117-3.3

Commit message: Finished schematic
Parts:
- added C1: 100n, Capacitor_SMD:C_0603_1608Metric, symbol Device:C
- added C10, C2: 18p, Capacitor_SMD:C_0402_1005Metric, symbol Device:C
- added C11, C14, C16, C17, C18, C19, C23, C3, C4, C5, C6, C9: 100n, Capacitor_SMD:C_0402_1005Metric, symbol Device:C
- added C15: 10u, Capacitor_SMD:C_0603_1608Metric, symbol Device:C
- added C24, C25: 10p, Capacitor_SMD:C_0402_1005Metric, symbol Device:C
- added C7, C8: 1u, Capacitor_SMD:C_0603_1608Metric, symbol Device:C
- added D2: YELLOW, LED_SMD:LED_0805_2012Metric, symbol Device:LED
- added D3, D4, D5, D6: WS2812B, LED_SMD:LED_WS2812B_PLCC4_5.0x5.0mm_P3.2mm, symbol LED:WS2812B
- added H1, H2, H3, H4: MountingHole, MountingHole:MountingHole_2.2mm_M2, symbol Mechanical:MountingHole
- added J5: USB_A, libs:USB-A-TH_USB-231-ARY, symbol Connector:USB_A
- added J7, J8: Conn_01x04_Pin, libs:HDR-TH_4P-P2.54-V-M, symbol Connector:Conn_01x04_Pin
- added R10: 12k, Resistor_SMD:R_0603_1608Metric, symbol Device:R
- added R11, R14, R15, R16, R4, R6, R7: 100k, Resistor_SMD:R_0603_1608Metric, symbol Device:R
- added R12, R13, R8: 56k, Resistor_SMD:R_0402_1005Metric, symbol Device:R
- added R17: 10k, Capacitor_SMD:C_0402_1005Metric, symbol Device:R
- added R18: 1k, Resistor_SMD:R_0603_1608Metric, symbol Device:R
- added R9: 1M, Resistor_SMD:R_0603_1608Metric, symbol Device:R
- added SW1: SW_SPDT, libs:SW-SMD_K3-1280S-K1, symbol Switch:SW_SPDT
- added TP1, TP3, TP4, TP5, TP6, TP7: TestPoint, TestPoint:TestPoint_THTPad_D1.5mm_Drill0.7mm, symbol Connector:TestPoint
- added U10: STM32F103C8T6, Package_QFP:LQFP-48_7x7mm_P0.5mm, symbol MCU_ST_STM32F1:STM32F103C8Tx
- added U3, U4, U5, U6, U8: USBLC6-2SC6, Package_TO_SOT_SMD:SOT-23-6, symbol Power_Protection:USBLC6-2SC6
- added U7, U9: MIC2026-1YM, Package_SO:SOIC-8_3.9x4.9mm_P1.27mm, symbol Power_Management:MIC2026-1xM
- added Y1: 24MHz, libs:CRYSTAL-SMD_4P-L3.2-W2.5-BL_SIT8008BI, symbol Device:Crystal_GND24
- added Y2: 16MHz, libs:OSC-SMD_4P-L3.2-W2.5-BL, symbol Device:Crystal_GND24
- R3: LCSC C25905 -> C25796
Connections:
- net +3V3: now also U1.10 (VDDA33), U1.15 (VDD33), U1.23 (VDD33), U1.29 (VDDA33), U1.36 (VDDA33), U1.5 (VDDA33), C1.1, C15.1, C16.1, C17.1, C18.1, C19.1, C3.1, C3.2, C4.1, C4.2, C5.1, C5.2, C6.1, C6.2, C7.1, C7.2, J7.4 (Pin_4), J8.4 (Pin_4), R11.2, SW1.1 (A), U10.1 (VBAT), U10.24 (VDD), U10.36 (VDD), U10.48 (VDD), U10.9 (VDDA)
- net GND: now also J2.A1 (GND), J2.A12 (GND), J2.B1 (GND), J2.B12 (GND), J2.S1 (SHIELD), J3.A1 (GND), J3.A12 (GND), J3.B1 (GND), J3.B12 (GND), J3.S1 (SHIELD), U1.11 (TEST), C1.2, C10.2, C11.2, C14.2, C15.2, C16.2, C17.2, C18.2, C19.2, C2.2, C23.2, C24.2, C25.2, C8.2, C9.2, D2.1 (K), D3.3 (VSS), D4.3 (VSS), D5.3 (VSS), D6.3 (VSS), J5.4 (GND), J5.5 (Shield), J7.1 (Pin_1), J8.1 (Pin_1), R10.1, R14.1, R15.1, R16.1, R4.1, R7.1, SW1.3 (C), U10.23 (VSS), U10.35 (VSS), U10.47 (VSS), U10.8 (VSSA), U3.2 (GND), U4.2 (GND), U5.2 (GND), U6.2 (GND), U7.6 (GND), U8.2 (GND), U9.6 (GND), Y1.2, Y1.4, Y2.2, Y2.4
- net UP_D+: now also U1.31 (USBDP_UP), U3.4 (I/O2); no longer J1.A6 (D+), J1.B6 (D+)
- net UP_D-: now also U1.30 (USBDM_UP), U3.6 (I/O1); no longer J1.A7 (D-), J1.B7 (D-)
- net VBUS: now also D3.1 (VDD), D4.1 (VDD), D5.1 (VDD), D6.1 (VDD), R6.2, TP1.1, U3.5 (VBUS), U7.7 (IN), U9.7 (IN)
- net VBUS_3: now reaches J4.1 (VBUS)
- net VBUS_3: now also TP6.1, U6.5 (VBUS), U9.8 (OUTA)
- net at J4.2 (D-): now also U6.3 (I/O2)
- net at J4.3 (D+): now also U6.1 (I/O1)
- net at R3.1: now also J3.A5 (CC1)
- net VBUS_2: now reaches R3.2
- net VBUS_2: now also J3.A4 (VBUS), J3.A9 (VBUS), J3.B4 (VBUS), J3.B9 (VBUS), R8.2, TP4.1, U5.5 (VBUS), U7.5 (OUTB)
- net VBUS_1: now reaches J2.A4 (VBUS), J2.A9 (VBUS), J2.B4 (VBUS), J2.B9 (VBUS)
- net VBUS_1: now also R12.2, R13.2, TP3.1, U4.5 (VBUS), U7.8 (OUTA)
- net at J2.A5 (CC1): now also R12.1
- net at J2.A6 (D+): now also J2.B6 (D+), U4.3 (I/O2)
- net at J2.A7 (D-): now also J2.B7 (D-), U4.1 (I/O1)
- net at J2.B5 (CC2): now also R13.1
- net DOWN_1_D-: now reaches U1.1 (USBDM_DN1/PRT_DIS_M1)
- net DOWN_1_D-: now also U4.6 (I/O1)
- net EN1: now reaches U1.12 (PRTPWR1/BC_EN1)
- net EN1: now also U10.25 (PB12), U7.1 (ENA)
- net OCS_N1: now reaches U1.13 (OCS_N1)
- net OCS_N1: now also U10.45 (PB8), U7.2 (FLGA)
- net at U1.14 (CRFILT): now also C11.1
- net EN2: now reaches U1.16 (PRTPWR2/BC_EN2)
- net EN2: now also U10.26 (PB13), U7.4 (ENB)
- net OCS_N2: now reaches U1.17 (OCS_N2)
- net OCS_N2: now also U10.46 (PB9), U7.3 (FLGB)
- net EN3: now reaches U1.18 (PRTPWR3/BC_EN3)
- net EN3: now also U10.27 (PB14), U9.1 (ENA)
- net OCS_N3: now reaches U1.19 (OCS_N3)
- net OCS_N3: now also U10.21 (PB10), U9.2 (FLGA)
- net DOWN_1_D+: now reaches U1.2 (USBDP_DN1/PRT_DIS_P1)
- net DOWN_1_D+: now also U4.4 (I/O2)
- net EN4: now reaches U1.20 (PRTPWR4/BC_EN4)
- net EN4: now also U10.28 (PB15), U9.4 (ENB)
- net OCS_N4: now reaches U1.21 (OCS_N4)
- net OCS_N4: now also U10.22 (PB11), U9.3 (FLGB)
- net at U1.22 (SDA/SMBDATA/NON_REM1): now also R15.2
- net at U1.24 (SCL/SMBCLK/CFG_SEL0): now also R16.2
- net at U1.25 (HS_IND/CFG_SEL1): now also R4.2
- net at U1.26 (RESET_N): now also C14.1, R11.1
- net at U1.27 (VBUS_DET): now also C8.1, R6.1, R7.2
- net at U1.28 (SUSP_IND/LOCAL_PWR/NON_REM0): now also R14.2
- net DOWN_2_D-: now reaches U1.3 (USBDM_DN2/PRT_DIS_M2)
- net DOWN_2_D-: now also U5.6 (I/O1)
- net at U1.32 (XTALOUT): now also C2.1, R9.1, Y1.3
- net at U1.33 (XTALIN/CLKIN): now also C10.1, R9.2, Y1.1
- net at U1.34 (PLLFILT): now also C9.1
- net at U1.35 (RBIAS): now also R10.2
- net DOWN_2_D+: now reaches U1.4 (USBDP_DN2/PRT_DIS_P2)
- net DOWN_2_D+: now also U5.4 (I/O2)
- net DOWN_3_D-: now reaches U1.6 (USBDM_DN3/PRT_DIS_M3)
- net DOWN_3_D-: now also U6.6 (I/O1)
- net DOWN_3_D+: now reaches U1.7 (USBDP_DN3/PRT_DIS_P3)
- net DOWN_3_D+: now also U6.4 (I/O2)
- net DOWN_4_D-: now reaches U1.8 (USBDM_DN4/PRT_DIS_M4)
- net DOWN_4_D-: now also U8.6 (I/O1)
- net DOWN_4_D+: now reaches U1.9 (USBDP_DN4/PRT_DIS_P4)
- net DOWN_4_D+: now also U8.4 (I/O2)
- net at J3.A6 (D+): now also J3.B6 (D+), U5.3 (I/O2)
- net at J3.A7 (D-): now also J3.B7 (D-), U5.1 (I/O1)
- net at J3.B5 (CC2): now also R8.1
- new net: J5.2 (D-), U8.3 (I/O2)
- new net: J5.3 (D+), U8.1 (I/O1)
- new net: D3.2 (DOUT), D4.4 (DIN)
- new net: D5.2 (DOUT), D6.4 (DIN)
- new net: J1.A7 (D-), J1.B7 (D-), U3.1 (I/O1)
- new net: J1.A6 (D+), J1.B6 (D+), U3.3 (I/O2)
- new net: D4.2 (DOUT), D5.4 (DIN)
- new net BOOT0: R17.2, U10.44 (BOOT0)
- new net DEBUG: R18.1, TP5.1, U10.2 (PC13)
- new net DEBUG_LED: D2.2 (A), R18.2
- new net HSE_IN: C24.1, U10.5 (PD0), Y2.1
- new net HSE_OUT: C25.1, U10.6 (PD1), Y2.3
- new net LED_DATA: D3.4 (DIN), U10.17 (PA7)
- new net NRST: C23.1, U10.7 (NRST)
- new net SWCLK: J8.2 (Pin_2), U10.37 (PA14)
- new net SWDIO: J8.3 (Pin_3), U10.34 (PA13)
- new net SW_BOOT0: R17.1, SW1.2 (B)
- new net USART_RX: J7.2 (Pin_2), U10.43 (PB7)
- new net USART_TX: J7.3 (Pin_3), U10.42 (PB6)
- new net VBUS_4: J5.1 (VBUS), TP7.1, U8.5 (VBUS), U9.5 (OUTB)
- no-connect marks 2 -> 26
Other:
- note added: "'Dumb' USB Type-A => power advertisement not required"
- note added: "1x 100nF per V_DD pin"
- note added: "7-bit I2C slave address = 0b1010000b."
- note added: "Advertise 5V/500mA sink"
- note added: "C_load = 2*(C_LO - C_S) = 2*(12-4) ~= 15pF"
- note added: "C_load = 2*(C_LO - C_S) = 2*(9-4) = 10pF"
- note added: "DFP 1 (Type-C)"
- note added: "DFP 2 (Type-C)"
- note added: "DFP 3 (Type-A)"
- note added: "DFP 4 (Type-A)"
- note added: "Downstream Ports"
- note added: "ESD Protection on D+/D-"
- note added: "HIGH => Bootloader mode LOW => Run-prog mode"
- note added: "I = V/R = (3.3-2.2)/1 = 1.1 mA"
- note added: "Load Switches"
- note added: "MCU Debug LED"
- note added: "MIC2026 => dual-channel high-side switch made for USB hub downstream ports. 1. Guarantees at least 500 mA continuous per port (to meet USB spec). Typical current limit is ~1.0 A (min 0.65 A, max 1.25 A). 2. In short-circuit, it enters a constant-current mode and holds around that limit."
- note added: "Microcontroller"
- note added: "Mounting Holes"
- note added: "One decoupling cap per VDD pin (4)"
- note added: "Output to WS2812B strip (4 LEDs) ->"
- note added: "Requeset 5V/3A sink"
- note added: "Serial Wire Debug"
- note added: "Simply to read ENx and thus appropriately driver WS2812Bs"
- note added: "Strapping Pin Notes (from datasheet): 1. NON_REM[1:0] = 00 => all ports are removable 2. CFG_SEL[1:0] = 00 => Default configuration: strap options enabled, self-powered operation enabled, individual power switching, individual over-current sensing"
- note added: "UART"
- note added: "USB 2.0 Full-Speed Hub (4 DFPs, 2 Type-C, 2 Type-A)"
- note added: "USB Type-C Receptacle (UFP/Host)"
- note added: "USB2514BI USB 2.0 Full-Speed Hub Controller"
- note added: "Up to 1A output, Cuz JLC basic lol"
- note added: "V_BUS from USB-C receptacle (5V)"
- note added: "WS2812B Port-Active LEDs"
- note added: "^ Not stricly necessary"
- note removed: "56k pull up lah. advertise as source up to 500mA usb 2.0 spec lah"
- note removed: "USB 2.0 FS Hub (3 DPs, 1 Type-A, 2 Type-C)"
- note removed: "Up to 1A output"
- note removed: "V_BUS from USB-C receptacle (5V nom.)"
- company: (none) -> Lachlan Cooke
- title: (none) -> USB 2.0 Full-Speed Hub (4 DFPs, 2 Type-C, 2 Type-A)
- moved on the sheet: C12, C13, D1, J1, J2, J4, R1, R2, R5, TP2, U1, U2

Commit message: Significant work on pcb
Parts:
- added C20, C21, C22: 100n, Capacitor_SMD:C_0402_1005Metric, symbol Device:C
- R10: footprint Resistor_SMD:R_0603_1608Metric -> Resistor_SMD:R_0402_1005Metric; LCSC C22790 -> C25752
- R11, R14, R15, R16, R4, R6, R7: footprint Resistor_SMD:R_0603_1608Metric -> Resistor_SMD:R_0402_1005Metric; LCSC C25803 -> C25741
Connections:
- net +3V3: now also C20.1, C21.1, C22.1; no longer C3.2, C4.2, C5.2, C6.2, C7.2
- net DOWN_1_D+: now also U8.4 (I/O2); no longer U4.4 (I/O2)
- net DOWN_1_D-: now also U8.6 (I/O1); no longer U4.6 (I/O1)
- net DOWN_3_D+: now also U4.4 (I/O2); no longer U6.4 (I/O2)
- net DOWN_3_D-: now also U4.6 (I/O1); no longer U6.6 (I/O1)
- net DOWN_4_D+: now also U6.4 (I/O2); no longer U8.4 (I/O2)
- net DOWN_4_D-: now also U6.6 (I/O1); no longer U8.6 (I/O1)
- net EN1: now also U7.4 (ENB); no longer U7.1 (ENA)
- net EN2: now also U7.1 (ENA); no longer U7.4 (ENB)
- net EN3: now also U9.4 (ENB); no longer U9.1 (ENA)
- net EN4: now also U9.1 (ENA); no longer U9.4 (ENB)
- net GND: now also C3.2, C4.2, C5.2, C6.2, C7.2, R6.1, C20.2, C21.2, C22.2; no longer R7.1
- net OCS_N1: now also U7.3 (FLGB); no longer U7.2 (FLGA)
- net OCS_N2: now also U7.2 (FLGA); no longer U7.3 (FLGB)
- net OCS_N3: now also U9.3 (FLGB); no longer U9.2 (FLGA)
- net OCS_N4: now also U9.2 (FLGA); no longer U9.3 (FLGB)
- net VBUS: now also R7.2; no longer R6.2
- net VBUS_1: now also J5.1 (VBUS), TP7.1, U7.5 (OUTB), U8.5 (VBUS); no longer J2.A4 (VBUS), J2.A9 (VBUS), J2.B4 (VBUS), J2.B9 (VBUS), R12.2, R13.2, TP3.1, U4.5 (VBUS), U7.8 (OUTA)
- net VBUS_2: now also U7.8 (OUTA); no longer U7.5 (OUTB)
- net VBUS_3: now also J2.A4 (VBUS), J2.A9 (VBUS), J2.B4 (VBUS), J2.B9 (VBUS), R12.2, R13.2, TP3.1, U4.5 (VBUS), U9.5 (OUTB); no longer J4.1 (VBUS), TP6.1, U6.5 (VBUS), U9.8 (OUTA)
- net VBUS_4: now also J4.1 (VBUS), TP6.1, U6.5 (VBUS), U9.8 (OUTA); no longer J5.1 (VBUS), TP7.1, U8.5 (VBUS), U9.5 (OUTB)
- net at J5.2 (D-): now also U8.1 (I/O1); no longer U8.3 (I/O2)
- net at J5.3 (D+): now also U8.3 (I/O2); no longer U8.1 (I/O1)
- net at C8.1, U1.27 (VBUS_DET): now also R6.2, R7.1; no longer R6.1, R7.2
- net at J4.2 (D-): now also U6.1 (I/O1); no longer U6.3 (I/O2)
- net at J4.3 (D+): now also U6.3 (I/O2); no longer U6.1 (I/O1)
- no-connect marks 26 -> 28
Other:
- moved on the sheet: C15, C3, C4, C5, C6, C7

Commit message: Significant work on pcb again
Connections:
- net OCS_N1: now also U10.40 (PB4); no longer U10.45 (PB8)
- net OCS_N2: now also U10.39 (PB3); no longer U10.46 (PB9)
- net OCS_N3: now also U10.31 (PA10); no longer U10.21 (PB10)
- net OCS_N4: now also U10.32 (PA11); no longer U10.22 (PB11)
Changed lines of the file:
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@@
 	)
 	(no_connect
+		(at 73.66 245.11)
+	)
+	(no_connect
 		(at 396.24 130.81)
 	)
@@
 	)
 	(no_connect
+		(at 73.66 242.57)
+	)
+	(no_connect
 		(at 46.99 120.65)
 	)
@@
 	)
 	(no_connect
-		(at 73.66 227.33)
-	)
-	(no_connect
 		(at 46.99 118.11)
 	)
 	(no_connect
-		(at 73.66 229.87)
-	)
-	(no_connect
 		(at 73.66 224.79)
 	)
@@
 	)
 	(no_connect
-		(at 109.22 217.17)
-	)
-	(no_connect
 		(at 109.22 201.93)
 	)
@@
 	)
 	(no_connect
+		(at 73.66 247.65)
+	)
+	(no_connect
 		(at 109.22 199.39)
 	)
@@
 	)
 	(no_connect
-		(at 109.22 219.71)
+		(at 73.66 232.41)
 	)
 	(no_connect
-		(at 73.66 232.41)
+		(at 73.66 240.03)
 	)
 	(no_connect
@@
 	(wire
 		(pts
-			(xy 189.23 57.15) (xy 186.69 57.15)
+			(xy 64.77 227.33) (xy 73.66 227.33)
 		)
 		(stroke
@@
 	(wire
 		(pts
-			(xy 358.14 121.92) (xy 367.03 121.92)
+			(xy 189.23 57.15) (xy 186.69 57.15)
 		)
 		(stroke
@@
 	(wire
 		(pts
-			(xy 181.61 57.15) (xy 186.69 57.15)
+			(xy 118.11 217.17) (xy 109.22 217.17)
 		)
 		(stroke
@@
 	(wire
 		(pts
-			(xy 62.23 54.61) (xy 68.58 54.61)
+			(xy 358.14 121.92) (xy 367.03 121.92)
 		)
 		(stroke
@@
 	(wire
 		(pts
-			(xy 100.33 135.89) (xy 100.33 139.7)
+			(xy 181.61 57.15) (xy 186.69 57.15)
 		)
 		(stroke
@@
 	(wire
 		(pts
-			(xy 53.34 167.64) (xy 64.77 167.64)
+			(xy 62.23 54.61) (xy 68.58 54.61)
 		)
 		(stroke
@@
 	(wire
 		(pts
-			(xy 292.1 195.58) (xy 300.99 195.58)
+			(xy 100.33 135.89) (xy 100.33 139.7)
 		)
 		(stroke
@@
 	(wire
 		(pts
-			(xy 125.73 120.65) (xy 125.73 121.92)
+			(xy 53.34 167.64) (xy 64.77 167.64)
 		)
 		(stroke
@@
 	(wire
 		(pts
-			(xy 300.99 227.33) (xy 316.23 227.33)
+			(xy 292.1 195.58) (xy 300.99 195.58)
 		)
 		(stroke
@@
 	(wire
 		(pts
-			(xy 109.22 104.14) (xy 109.22 105.41)
+			(xy 125.73 120.65) (xy 125.73 121.92)
 		)
 		(stroke
@@
 	(wire
 		(pts
-			(xy 64.77 240.03) (xy 73.66 240.03)
+			(xy 300.99 227.33) (xy 316.23 227.33)
 		)
 		(stroke
@@
 	(wire
 		(pts
-			(xy 58.42 199.39) (xy 58.42 196.85)
+			(xy 109.22 104.14) (xy 109.22 105.41)
 		)
 		(stroke
@@
 	(wire
 		(pts
-			(xy 64.77 245.11) (xy 73.66 245.11)
+			(xy 58.42 199.39) (xy 58.42 196.85)
 		)
 		(stroke
@@
 	(wire
 		(pts
+			(xy 118.11 219.71) (xy 109.22 219.71)
+		)
+		(stroke
+			(width 0)
+			(type default)
+		)
+	)
+	(wire
+		(pts
 			(xy 358.14 95.25) (xy 358.14 121.92)
 		)
@@
 	(wire
 		(pts
+			(xy 64.77 229.87) (xy 73.66 229.87)
+		)
+		(stroke
+			(width 0)
+			(type default)
+		)
+	)
+	(wire
+		(pts
 			(xy 53.34 234.95) (xy 73.66 234.95)
 		)
@@
 	(wire
 		(pts
-			(xy 64.77 247.65) (xy 73.66 247.65)
-		)
-		(stroke
-			(width 0)
-			(type default)
-		)
-	)
-	(wire
-		(pts
 			(xy 300.99 195.58) (xy 316.23 195.58)
 		)
@@
 	(wire
 		(pts
-			(xy 64.77 242.57) (xy 73.66 242.57)
-		)
-		(stroke
-			(width 0)
-			(type default)
-		)
-	)
-	(wire
-		(pts
 			(xy 292.1 208.28) (xy 292.1 209.55)
 		)
@@
 		)
 	)
+	(label "OCS_N1"
+		(at 64.77 229.87 0)
+		(effects
+			(font
+				(size 1.27 1.27)
+			)
+			(justify left bottom)
+		)
+	)
 	(label "DOWN_3_D-"
 		(at 223.52 100.33 180)
@@
 		)
 	)
-	(label "OCS_N1"
-		(at 64.77 240.03 0)
-		(effects
-			(font
-				(size 1.27 1.27)
-			)
-			(justify left bottom)
-		)
-	)
 	(label "UP_D-"
 		(at 85.09 105.41 180)
@@
 		)
 	)
-	(label "OCS_N4"
-		(at 64.77 247.65 0)
-		(effects
-			(font
-				(size 1.27 1.27)
-			)
-			(justify left bottom)
-		)
-	)
 	(label "DOWN_3_D-"
 		(at 260.35 106.68 0)
@@
 		)
 	)
-	(label "OCS_N2"
-		(at 64.77 242.57 0)
-		(effects
-			(font
-				(size 1.27 1.27)
-			)
-			(justify left bottom)
-		)
-	)
 	(label "USART_RX"
 		(at 63.5 237.49 0)
@@
 		)
 	)
+	(label "OCS_N3"
+		(at 118.11 217.17 180)
+		(effects
+			(font
+				(size 1.27 1.27)
+			)
+			(justify right bottom)
+		)
+	)
 	(label "HSE_OUT"
 		(at 66.04 204.47 0)
@@
 		)
 	)
-	(label "OCS_N3"
-		(at 64.77 245.11 0)
-		(effects
-			(font
-				(size 1.27 1.27)
-			)
-			(justify left bottom)
-		)
-	)
 	(label "EN1"
 		(at 219.71 80.01 180)
@@
 		)
 	)
+	(label "OCS_N2"
+		(at 64.77 227.33 0)
+		(effects
+			(font
+				(size 1.27 1.27)
+			)
+			(justify left bottom)
+		)
+	)
 	(label "DOWN_4_D-"
 		(at 223.52 113.03 180)
@@
 		)
 	)
+	(label "OCS_N4"
+		(at 118.11 219.71 180)
+		(effects
+			(font
+				(size 1.27 1.27)
+			)
+			(justify right bottom)
+		)
+	)

Commit message: Board finished, sending out for fab
Parts:
- added SW2: SW_Push, libs:SW-SMD_L3.9-W3.0-P4.45, symbol Switch:SW_Push
Connections:
- net GND: now also SW2.1
- net NRST: now also SW2.2
Other:
- note added: "NRST has internal pull-up"
Changed lines of the file:
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@@
 		)
 	)
+	(text "NRST has internal pull-up"
+		(exclude_from_sim no)
+		(at 21.59 189.23 0)
+		(effects
+			(font
+				(size 0.762 0.762)
+				(thickness 0.254)
+				(bold yes)
+			)
+			(justify left top)
+		)
+	)
 	(text "'Dumb' USB Type-A => power advertisement not required"
 		(exclude_from_sim no)
@@
 	)
 	(junction
+		(at 19.05 203.2)
+		(diameter 0)
+		(color 0 0 0 0)
+	)
+	(junction
 		(at 232.41 55.88)
 		(diameter 0)
@@
 	)
 	(junction
+		(at 30.48 191.77)
+		(diameter 0)
+		(color 0 0 0 0)
+	)
+	(junction
 		(at 173.99 57.15)
 		(diameter 0)
@@
 	(wire
 		(pts
-			(xy 30.48 200.66) (xy 30.48 201.93)
+			(xy 30.48 200.66) (xy 30.48 203.2)
 		)
 		(stroke
@@
 	(wire
 		(pts
+			(xy 19.05 191.77) (xy 30.48 191.77)
+		)
+		(stroke
+			(width 0)
+			(type default)
+		)
+	)
+	(wire
+		(pts
 			(xy 39.37 213.36) (xy 34.29 213.36)
 		)
@@
 	(wire
 		(pts
+			(xy 19.05 204.47) (xy 19.05 203.2)
+		)
+		(stroke
+			(width 0)
+			(type default)
+		)
+	)
+	(wire
+		(pts
 			(xy 30.48 234.95) (xy 30.48 237.49)
 		)
@@
 	(wire
 		(pts
+			(xy 19.05 203.2) (xy 19.05 201.93)
+		)
+		(stroke
+			(width 0)
+			(type default)
+		)
+	)
+	(wire
+		(pts
 			(xy 212.09 54.61) (xy 212.09 55.88)
 		)
@@
 	(wire
 		(pts
+			(xy 19.05 203.2) (xy 30.48 203.2)
+		)
+		(stroke
+			(width 0)
+			(type default)
+		)
+	)
+	(wire
+		(pts
 			(xy 388.62 138.43) (xy 388.62 139.7)
 		)
@@
 	(symbol
 		(lib_id "power:GND")
-		(at 30.48 201.93 0)
+		(at 19.05 204.47 0)
 		(unit 1)
 		(exclude_from_sim no)
@@
 		(fields_autoplaced yes)
 		(property "Reference" "#PWR041"
-			(at 30.48 208.28 0)
+			(at 19.05 210.82 0)
 			(effects
 				(font
@@
 		)
 		(property "Value" "GND"
-			(at 30.48 207.01 0)
+			(at 19.05 209.55 0)
 			(effects
 				(font
@@
 		)
 		(property "Footprint" ""
-			(at 30.48 201.93 0)
+			(at 19.05 204.47 0)
 			(effects
 				(font
@@
 		)
 		(property "Datasheet" ""
-			(at 30.48 201.93 0)
+			(at 19.05 204.47 0)
 			(effects
 				(font
@@
 		)
 		(property "Description" "Power symbol creates a global label with name \"GND\" , ground"
-			(at 30.48 201.93 0)
+			(at 19.05 204.47 0)
 			(effects
 				(font
@@
 					(unit 1)
 				)
+			)
+		)
+	)
+	(symbol
+		(lib_id "Switch:SW_Push")
+		(at 19.05 196.85 90)
+		(unit 1)
+		(exclude_from_sim no)
+		(in_bom yes)
+		(on_board yes)
+		(dnp no)
+		(property "Reference" "SW2"
+			(at 20.32 195.5799 90)
+			(effects
+				(font
+					(size 1.27 1.27)
+				)
+				(justify right)
+			)
+		)
+		(property "Value" "SW_Push"
+			(at 20.32 199.39 90)
+			(effects
+				(font
+					(size 1.27 1.27)
+				)
+				(justify right)
+			)
+		)
+		(property "Footprint" "libs:SW-SMD_L3.9-W3.0-P4.45"
+			(at 13.97 196.85 0)
+			(effects
+				(font
+					(size 1.27 1.27)
+				)
+				(hide yes)
+			)
+		)
+		(property "Datasheet" "~"
+			(at 13.97 196.85 0)
+			(effects
+				(font
+					(size 1.27 1.27)
+				)
+				(hide yes)
+			)
+		)
+		(property "Description" "Push button switch, generic, two pins"
+			(at 19.05 196.85 0)
+			(effects
+				(font
+					(size 1.27 1.27)
+				)
+				(hide yes)
+			)
+		)
+		(property "LCSC" "C720477"
+			(at 19.05 196.85 90)
+			(effects
+				(font
+					(size 1.27 1.27)
+				)
+				(hide yes)
+			)
+		)
+		(pin "2"
+		)
+		(pin "1"
+		)
+		(instances
+			(project ""
+				(path "/70085d1f-377c-415d-a552-14e05032eb0b"
+					(reference "SW2")
+					(unit 1)
+				)

Commit message: Fixed erroneous LSCS part number (0603 instead of 0402)
Parts:
- C11, C14, C20, C21, C3, C4, C5, C6, C9: LCSC C14663 -> C1525
Changed lines of the file:
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@@
 			)
 		)
-		(property "LCSC" "C14663"
+		(property "LCSC" "C1525"
 			(at 137.16 115.57 0)
 			(effects
@@
 			)
 		)
-		(property "LCSC" "C14663"
+		(property "LCSC" "C1525"
 			(at 106.68 88.9 0)
 			(effects
@@
 			)
 		)
-		(property "LCSC" "C14663"
+		(property "LCSC" "C1525"
 			(at 125.73 115.57 0)
 			(effects
@@
 			)
 		)
-		(property "LCSC" "C14663"
+		(property "LCSC" "C1525"
 			(at 181.61 50.8 0)
 			(effects
@@
 			)
 		)
-		(property "LCSC" "C14663"
+		(property "LCSC" "C1525"
 			(at 201.93 50.8 0)
 			(effects
@@
 			)
 		)
-		(property "LCSC" "C14663"
+		(property "LCSC" "C1525"
 			(at 232.41 50.8 0)
 			(effects
@@
 			)
 		)
-		(property "LCSC" "C14663"
+		(property "LCSC" "C1525"
 			(at 191.77 50.8 0)
 			(effects
@@
 			)
 		)
-		(property "LCSC" "C14663"
+		(property "LCSC" "C1525"
 			(at 222.25 50.8 0)
 			(effects
@@
 			)
 		)
-		(property "LCSC" "C14663"
+		(property "LCSC" "C1525"
 			(at 212.09 50.8 0)
 			(effects
